Commit message: basic urdf structure + color/inertial macros

File: src/trailblazerml/dependencies/macros/colors.xacro (robot description, xacro)
@@ -1,15 +1,23 @@
 <?xml version="1.0"?>
 <robot xmlns:xacro="http://www.ros.org/wiki/xacro">
-    <material name="white">
-        <color rgba="1 1 1 1"/>
-    </material>
-    <material name="orange">
-        <color rgba="1 0.3 0.1 1"/>
-    </material>
-    <material name="blue">
-        <color rgba="0.2 0.2 1 1"/>
-    </material>
-    <material name="black">
-        <color rgba="0 0 0 1"/>
-    </material>
+    <!-- Define color materials -->
+    <xacro:macro name="material_color" params="color_name">
+        <xacro:choose>
+            <xacro:when value="${color_name == 'white'}">
+                1 1 1 1
+            </xacro:when>
+            <xacro:when value="${color_name == 'orange'}">
+                1 0.3 0.1 1
+            </xacro:when>
+            <xacro:when value="${color_name == 'blue'}">
+                0.2 0.2 1 1
+            </xacro:when>
+            <xacro:when value="${color_name == 'black'}">
+                0 0 0 1
+            </xacro:when>
+            <xacro:otherwise>
+                1 1 1 1  <!-- Default to white if no match -->
+            </xacro:otherwise>
+        </xacro:choose>
+    </xacro:macro>
 </robot>
