Commit message: first xacro rover project

File: src/trailblazerml/description/parts/wheel_right.xacro (robot description, xacro)
@@ -1,7 +1,9 @@
+<?xml version="1.0"?>
+<robot xmlns:xacro="http://www.ros.org/wiki/xacro" >
 <xacro:macro name="wheel" params="name mass">
         <link name="${name}">
             <visual>
                 <geometry>
-                    <cylinder radius="${wheel_radius}" length="${wheel_length}" />
+                     <mesh filename="file://$(find trailblazerml)/models/rover_stl/wheel_right.stl" scale="1 1 1"/>
                 </geometry>
                 <material name="${wheel_color_name}">
@@ -11,5 +13,5 @@
             <collision>
                 <geometry>
-                    <cylinder length="${wheel_length}" radius="${wheel_radius}" />/>
+                     <mesh filename="file://$(find trailblazerml)/models/rover_stl/wheel_right.stl" scale="1 1 1"/>
                 </geometry>
                 <material name="blue"/>
@@ -20,2 +22,3 @@
         </link>
     </xacro:macro>
+</robot>
