Commit message: refactor wheel_left.xacro

File: src/trailblazerml/description/parts/wheel_left.xacro (robot description, xacro)
@@ -1,18 +1,19 @@
 <?xml version="1.0"?>
-<robot xmlns:xacro="http://www.ros.org/wiki/xacro" >
-<xacro:macro name="wheel" params="name mass">
+<robot xmlns:xacro="http://www.ros.org/wiki/xacro">
+    <xacro:include filename="../macros/colors.xacro" />
+    <xacro:include filename="../macros/inertial_macros.xacro" />
+    <xacro:property name="wheel_color_name" value="blue" />
+    <xacro:property name="wheel_color_rgb" value="${xacro:call('material_color', wheel_color_name)}" />
+    <xacro:macro name="wheel_left" params="name mass">
         <link name="${name}">
             <visual>
-                <origin xyz="0.12 0.055 0" rpy="0 0 ${pi/2}"/>
+                <origin xyz="0.6 0.07 -0.17" rpy="${pi/2} ${pi/2} ${pi/2}"/>
                 <geometry>
-                     <mesh filename="file://$(find trailblazerml)/models/rover_stl/wheel_left.stl" scale="1 1 1"/>
+                    <mesh filename="file://$(find trailblazerml)/models/rover_stl/wheel_left.stl" scale="0.001 0.001 0.001"/>
                 </geometry>
-                <material name="${wheel_color_name}">
-                    <color rgba="${wheel_color_rgb}"/>
-                </material>
             </visual>
             <collision>
                 <geometry>
-                     <mesh filename="file://$(find trailblazerml)/models/rover_stl/wheel_left.stl" scale="1 1 1"/>
+                    <mesh filename="file://$(find trailblazerml)/models/rover_stl/wheel_left.stl" scale="1 1 1"/>
                 </geometry>
                 <material name="blue"/>
@@ -22,4 +23,10 @@
             </xacro:inertial_cylinder>
         </link>
+        <!-- Fix the joint definition with proper quotes -->
+        <joint name="${name}_joint" type="continuous">
+            <parent link="rover_body"/>
+            <child link="${name}"/>
+            <origin xyz="0 0 0"/>
+        </joint>
     </xacro:macro>
 </robot>

File: src/trailblazerml/description/parts/wheel_right.xacro (robot description, xacro)
@@ -1,5 +1,5 @@
 <?xml version="1.0"?>
 <robot xmlns:xacro="http://www.ros.org/wiki/xacro" >
-<xacro:macro name="wheel" params="name mass">
+<xacro:macro name="wheel_right" params="name mass">
         <link name="${name}">
             <visual>

File: src/trailblazerml/description/robot.urdf.xacro (robot description, xacro)
@@ -1,5 +1,10 @@
-<?xml version=1.0>
+<?xml version="1.0"?>
 <robot xmlns:xacro="http://www.ros.org/wiki/xacro"  name="rover">
     <!--  Tutaj wszystkie importy części łazika -->
-    <!-- -------------------------------------- -->
+        <xacro:include filename="robot_core.xacro" />
+        <xacro:include filename="parts/wheel_left.xacro" />
+        <xacro:include filename="parts/wheel_right.xacro" />
+    <!--  wywołanie kół -->
+        <xacro:wheel_left name="wheel_left_front" mass="0.5">
+        </xacro:wheel_left>
 </robot>

File: src/trailblazerml/description/robot_core.xacro (robot description, xacro)
@@ -1,12 +1,7 @@
 <?xml version="1.0"?>
-<robot xmlns:xacro="http://www.ros.org/wiki/xacro">
+<robot xmlns:xacro="http://www.ros.org/wiki/xacro" >
     <!-- IMPORTY CZĘŚCI -->
         <xacro:include filename="macros/colors.xacro" />
         <xacro:include filename="macros/inertial_macros.xacro" />
-        <xacro:include filename="parts/wheel_left.xacro" />
-        <xacro:include filename="parts/wheel_right.xacro" />
-        <xacro:include filename="parts/camera.xacro" />
-        <xacro:include filename="parts/depth_camera.xacro" />
-    <!-- -------------------------------------- -->
     <!-- DEFINIOWANIE STAŁYCH -->
         <xacro:property name="wheel_radius" value="0.04" />
@@ -14,10 +9,8 @@
         <xacro:property name="wheel_color_name" value="red" />
         <xacro:property name="wheel_color_rgb" value="${xacro:call('material_color', wheel_color_name)}" />
-    <!-- -------------------------------------- -->
     <!-- BASE LINK - STAŁY LINK DO KTÓREGO BĘDĄ PODŁĄCZONE WSZYSTKIE CZĘŚCI -->
     <!-- NIE JEST ON RUCHOMY, NIC W NIM NIE DEFINIUJEMY, POTRZEBY DO ODOM PÓŹNIEJ -->
         <link name="base_link">
         </link>
-    <!-- -------------------------------------- -->
     <joint name="rover_body_joint" type="fixed">
         <parent link="base_link" />
@@ -28,7 +21,7 @@
         <link name="rover_body">
             <visual>
-                <origin xyz="0 0 0" rpy="0 0 0" />
+                <origin xyz="0 0 0" rpy="${pi/2} 0 0" />
                 <geometry>
-                    <mesh filename="file://$(find trailblazerml)/models/rover_stl/body.stl" scale="1 1 1"/>
+                    <mesh filename="file://$(find trailblazerml)/models/rover_stl/body.stl" scale="0.001 0.001 0.001"/>
                 </geometry>
             </visual>
@@ -36,5 +29,5 @@
                 <origin xyz="0 0 0" rpy="0 0 0" />
                 <geometry>
-                    <box size="1 1 1">
+                    <box size="0.5 0.5 0.5" />
                 </geometry>
             </collision>
@@ -43,4 +36,3 @@
             </xacro:inertial_box>
         </link>
-    <!-- -------------------------------------- -->
 </robot>
