Commit message: make new structure of package gazebo_rviz

File: src/trailblazerml/dependencies/robot.urdf.xacro (robot description, xacro)
@@ -1,5 +1,38 @@
 <?xml version=1.0>
 <robot xmlns:xacro="http://www.ros.org/wiki/xacro"  name="rover">
-    <!--  Tutaj wszystkie importy części łazika -->
-    <!-- -------------------------------------- -->
+    <!-- Import color definitions -->
+    <xacro:include filename="macros/colors.xacro"/>
+    <!-- Import inertial macros -->
+    <xacro:include filename="macros/inertial_macros.xacro"/>
+    <!-- Base link -->
+    <link name="base_link">
+        <visual>
+            <geometry>
+                <box size="1 1 0.5"/>
+            </geometry>
+            <material name="orange"/>
+        </visual>
+        <collision>
+            <geometry>
+                <box size="1 1 0.5"/>
+            </geometry>
+        </collision>
+        <xacro:inertial_macro mass="10" ixx="1" iyy="1" izz="1"/>
+    </link>
+    <!-- Wheel links -->
+    <link name="wheel_front_left">
+        <visual>
+            <geometry>
+                <cylinder length="0.1" radius="0.2"/>
+            </geometry>
+            <material name="black"/>
+        </visual>
+        <collision>
+            <geometry>
+                <cylinder length="0.1" radius="0.2"/>
+            </geometry>
+        </collision>
+        <xacro:inertial_macro mass="1" ixx="0.1" iyy="0.1" izz="0.1"/>
+    </link>
+    <!-- Add more wheels and joints as needed -->
 </robot>
