Commit message: new controller - odom and base link static

File: src/gazebo_viz/description/camera.xacro (robot description, xacro)
@@ -10,4 +10,11 @@
             <geometry>
                 <box size="0.010 0.03 0.03"/>
+            </geometry>
+            <material name="black"/>
+        </visual>
+        <visual>
+            <origin xyz="0 0 -0.05"/>
+            <geometry>
+                <cylinder radius="0.002" length="0.1"/>
             </geometry>
             <material name="black"/>
@@ -27,5 +34,4 @@
             <update_rate>10</update_rate>
             <camera>
-                <camera_info_topic>camera/camera_info</camera_info_topic>
                 <horizontal_fov>1.089</horizontal_fov>
                 <image>
@@ -39,6 +45,7 @@
                 </clip>
             </camera>
-            <topic>camera/image_raw</topic>
-            <gz_frame_id>camera_link_optical</gz_frame_id>
+            <plugin name="camera_controller" filename="libgazebo_ros_camera.so">
+                <frame_name>camera_link_optical</frame_name>
+            </plugin>
         </sensor>
     </gazebo>

File: src/gazebo_viz/description/depth_camera.xacro (robot description, xacro)
@@ -4,5 +4,5 @@
         <parent link="chassis"/>
         <child link="camera_link"/>
-        <origin xyz="0.305 0 0.08" rpy="0 0 0"/>
+        <origin xyz="0.4 0.01 -0.01" rpy="0 0.18 0"/>
     </joint>
     <link name="camera_link">

File: src/gazebo_viz/description/gazebo_control.xacro (robot description, xacro)
@@ -3,5 +3,5 @@
     <gazebo>
         <plugin name="differential_drive_controller" filename="libgazebo_ros_diff_drive.so">
-            <num_wheel_pairs>2</num_wheel_pairs>
+            <num_wheel_pairs>4</num_wheel_pairs>
             <left_joint>left_wheel_front_joint</left_joint>
             <left_joint>left_wheel_back_joint</left_joint>

File: src/gazebo_viz/description/robot.urdf.xacro (robot description, xacro)
@@ -2,6 +2,7 @@
 <robot xmlns:xacro="http://www.ros.org/wiki/xacro"  name="my_robot">
     <xacro:include filename="robot_core.xacro" />
-    <xacro:include filename="camera.xacro" />
-    <!--<xacro:include filename="gazebo_control.xacro" /> -->
+    <!--<xacro:include filename="camera.xacro" /> -->
+    <xacro:include filename="depth_camera.xacro" />
+    <xacro:include filename="gazebo_control.xacro" />
     <xacro:include filename="ros2_control.xacro" />
 </robot>
