Commit message: mapping

File: src/gazebo_viz/description/depth_camera.xacro (robot description, xacro)
@@ -4,5 +4,5 @@
         <parent link="chassis"/>
         <child link="camera_link"/>
-        <origin xyz="0.4 0.01 -0.01" rpy="0 0.18 0"/>
+        <origin xyz="0.4 0.01 -0.01" rpy="0 0.0 0"/>
     </joint>
     <link name="camera_link">
@@ -23,7 +23,7 @@
         <material>Gazebo/Red</material>
         <sensor name="camera" type="depth">
-            <pose> 0 0 0 0 0 0 </pose>
+            <pose> 0 0 0 0 0 1 </pose>
             <visualize>true</visualize>
-            <update_rate>10</update_rate>
+            <update_rate>1</update_rate>
             <camera>
                 <horizontal_fov>1.089</horizontal_fov>
