Commit message: working nav

File: src/trailblazer_description/description/robot.urdf.xacro (robot description, xacro)
@@ -1,8 +1,15 @@
 <?xml version="1.0"?>
 <robot xmlns:xacro="http://www.ros.org/wiki/xacro"  name="my_robot">
+    <xacro:arg name="use_ros2_control" default="true"/>
+    <xacro:arg name="sim_mode" default="false"/>
     <xacro:include filename="robot_core.xacro" />
     <xacro:include filename="lidar.xacro" />
     <!--<xacro:include filename="camera.xacro" /> -->
     <xacro:include filename="depth_camera.xacro" />
-    <xacro:include filename="ros2_control.xacro" />
+    <xacro:if value="$(arg use_ros2_control)">
+        <xacro:include filename="ros2_control.xacro" />
+    </xacro:if>
+    <xacro:unless value="$(arg use_ros2_control)">
+        <xacro:include filename="ros2_control_gazebo.xacro" />
+    </xacro:unless>
 </robot>

File: src/trailblazer_description/description/robot_core.xacro (robot description, xacro)
@@ -55,5 +55,5 @@
             <origin xyz="0 0 0.1"/>
             <geometry>
-                <box size="${chassis_length/2} ${chassis_width/2} ${chassis_height/2}"/>
+                <box size="${chassis_length} ${chassis_width} ${chassis_height}"/>
             </geometry>
         </collision>

File: src/trailblazer_description/description/ros2_control.xacro (robot description, xacro)
@@ -13,6 +13,6 @@
         <joint name="left_wheel_front_joint">
         <command_interface name="velocity">
-            <param name="min">-3</param>
-            <param name="max">3</param>
+            <param name="min">-0.5</param>
+            <param name="max">0.5</param>
         </command_interface>
         <state_interface name="position" />
@@ -21,6 +21,6 @@
         <joint name="right_wheel_front_joint">
             <command_interface name="velocity">
-                <param name="min">-3</param>
-                <param name="max">3</param>
+                <param name="min">-0.5</param>
+                <param name="max">0.5</param>
             </command_interface>
             <state_interface name="velocity" />
@@ -29,6 +29,6 @@
         <joint name="left_wheel_back_joint">
         <command_interface name="velocity">
-            <param name="min">-3</param>
-            <param name="max">3</param>
+            <param name="min">-0.5</param>
+            <param name="max">0.5</param>
         </command_interface>
         <state_interface name="position" />
@@ -37,6 +37,6 @@
         <joint name="right_wheel_back_joint">
             <command_interface name="velocity">
-                <param name="min">-3</param>
-                <param name="max">3</param>
+                <param name="min">-0.5</param>
+                <param name="max">0.5</param>
             </command_interface>
             <state_interface name="velocity" />

File: src/trailblazer_description/description/ros2_control_gazebo.xacro (robot description, xacro)
@@ -40,5 +40,5 @@
     <gazebo>
         <plugin name="gazebo_ros2_control" filename="libgazebo_ros2_control.so">
-            <parameters>$(find trailblazer_wheels)/config/controllers.yaml</parameters>
+            <parameters>$(find trailblazer_gazebo)/config/controllers.yaml</parameters>
         </plugin>
     </gazebo>
