Commit message: update slam

File: src/trailblazer_description/urdf/gps.xacro (robot description, xacro)
@@ -18,5 +18,22 @@
           <!-- ensure the sensor is active (required) -->
           <always_on>true</always_on>
-          <update_rate>30</update_rate>
+          <update_rate>1</update_rate>
+          <pose>0 0 0 0 0 0</pose>
+          <gps>
+            <position_sensing>
+              <horizontal>
+                <noise type="gaussian">
+                  <mean>0.0</mean>
+                  <stddev>0.01</stddev>
+                </noise>
+              </horizontal>
+              <vertical>
+                <noise type="gaussian">
+                  <mean>0.0</mean>
+                  <stddev>0.01</stddev>
+                </noise>
+              </vertical>
+            </position_sensing>
+          </gps>
           <plugin name="gps" filename="libgazebo_ros_gps_sensor.so">
             <ros>

File: src/trailblazer_description/urdf/imu.xacro (robot description, xacro)
@@ -17,15 +17,54 @@
         <gravity>true</gravity>
         <sensor name="imu_sensor" type="imu">
+        <always_on>true</always_on>
+          <update_rate>200</update_rate>
+          <imu>
+            <angular_velocity>
+              <x>
+                <noise type="gaussian">
+                  <mean>0.0</mean>
+                  <stddev>2e-4</stddev>
+                </noise>
+              </x>
+              <y>
+                <noise type="gaussian">
+                  <mean>0.0</mean>
+                  <stddev>2e-4</stddev>
+                </noise>
+              </y>
+              <z>
+                <noise type="gaussian">
+                  <mean>0.0</mean>
+                  <stddev>2e-4</stddev>
+                </noise>
+              </z>
+            </angular_velocity>
+            <linear_acceleration>
+              <x>
+                <noise type="gaussian">
+                  <mean>0.0</mean>
+                  <stddev>1.7e-2</stddev>
+                </noise>
+              </x>
+              <y>
+                <noise type="gaussian">
+                  <mean>0.0</mean>
+                  <stddev>1.7e-2</stddev>
+                </noise>
+              </y>
+              <z>
+                <noise type="gaussian">
+                  <mean>0.0</mean>
+                  <stddev>1.7e-2</stddev>
+                </noise>
+              </z>
+            </linear_acceleration>
+          </imu>
            <plugin filename="libgazebo_ros_imu_sensor.so" name="imu_plugin">
+              <initial_orientation_as_reference>false</initial_orientation_as_reference>
               <ros>
                 <namespace>/imu</namespace>
                 <remapping>~/out:=data</remapping>
               </ros>
-              <alwaysOn>true</alwaysOn>
-              <bodyName>base_link</bodyName>
-              <topicName>imu</topicName>
-              <serviceName>imu_service</serviceName>
-              <gaussianNoise>0.0</gaussianNoise>
-              <updateRate>20.0</updateRate>
             </plugin>
         </sensor>

File: src/trailblazer_description/urdf/rover.urdf.xacro (robot description, xacro)
@@ -45,5 +45,5 @@
       <parent link="base_link"/>
       <child link="chassis"/>
-      <origin xyz="0 0 0" rpy="1.5708 0 1.5708"/>
+      <origin xyz="0 0 0.365" rpy="1.5708 0 1.5708"/>
   </joint>
   <link
@@ -51,5 +51,5 @@
     <inertial>
       <origin
-        xyz="0.00322150223165306 -0.0317835441688463 0.0392262662545424"
+        xyz="0.00322150223165306 -0.0317835441688463 0.404226266"
         rpy="0 0 0" />
       <mass
