Commit message: kalman jednak nie działa :c

File: src/trailblazer_description/urdf/imu.xacro (robot description, xacro)
@@ -17,69 +17,17 @@
         <gravity>true</gravity>
         <sensor name="imu_sensor" type="imu">
-   <plugin filename="libgazebo_ros_imu_sensor.so" name="imu_plugin">
-      <ros>
-        <namespace>/imu</namespace>
-        <remapping>~/out:=data</remapping>
-      </ros>
-      <initial_orientation_as_reference>false</initial_orientation_as_reference>
-    </plugin>
-    <always_on>true</always_on>
-    <update_rate>100</update_rate>
-    <visualize>true</visualize>
-    <imu>
-      <angular_velocity>
-        <x>
-          <noise type="gaussian">
-            <mean>0.0</mean>
-            <stddev>2e-4</stddev>
-            <bias_mean>0.0000075</bias_mean>
-            <bias_stddev>0.0000008</bias_stddev>
-          </noise>
-        </x>
-        <y>
-          <noise type="gaussian">
-            <mean>0.0</mean>
-            <stddev>2e-4</stddev>
-            <bias_mean>0.0000075</bias_mean>
-            <bias_stddev>0.0000008</bias_stddev>
-          </noise>
-        </y>
-        <z>
-          <noise type="gaussian">
-            <mean>0.0</mean>
-            <stddev>2e-4</stddev>
-            <bias_mean>0.0000075</bias_mean>
-            <bias_stddev>0.0000008</bias_stddev>
-          </noise>
-        </z>
-      </angular_velocity>
-      <linear_acceleration>
-        <x>
-          <noise type="gaussian">
-            <mean>0.0</mean>
-            <stddev>1.7e-2</stddev>
-            <bias_mean>0.1</bias_mean>
-            <bias_stddev>0.001</bias_stddev>
-          </noise>
-        </x>
-        <y>
-          <noise type="gaussian">
-            <mean>0.0</mean>
-            <stddev>1.7e-2</stddev>
-            <bias_mean>0.1</bias_mean>
-            <bias_stddev>0.001</bias_stddev>
-          </noise>
-        </y>
-        <z>
-          <noise type="gaussian">
-            <mean>0.0</mean>
-            <stddev>1.7e-2</stddev>
-            <bias_mean>0.1</bias_mean>
-            <bias_stddev>0.001</bias_stddev>
-          </noise>
-        </z>
-      </linear_acceleration>
-    </imu>
-  </sensor>
+           <plugin filename="libgazebo_ros_imu_sensor.so" name="imu_plugin">
+              <ros>
+                <namespace>/imu</namespace>
+                <remapping>~/out:=data</remapping>
+              </ros>
+              <alwaysOn>true</alwaysOn>
+              <bodyName>base_footprint</bodyName>
+              <topicName>imu</topicName>
+              <serviceName>imu_service</serviceName>
+              <gaussianNoise>0.0</gaussianNoise>
+              <updateRate>20.0</updateRate>
+            </plugin>
+        </sensor>
     </gazebo>
 </robot>

File: src/trailblazer_description/urdf/rover.urdf.xacro (robot description, xacro)
@@ -2,5 +2,4 @@
 <robot name="legendary_rover" xmlns:xacro="http://www.ros.org/wiki/xacro">
   <!-- ******************************* XACRO ******************************* -->
-  <xacro:include filename="depth_camera.xacro" />
   <xacro:include filename="lidar.xacro" />
   <xacro:include filename="imu.xacro" />
@@ -10,8 +9,34 @@
   <xacro:if value="$(arg use_ros2_control)">
       <xacro:include filename="ros2_control.xacro" />
+      <!-- ******************************* OAK-D START ******************************* -->
+      <xacro:arg name="camera_name" default="oak" />
+      <xacro:arg name="camera_model" default="OAK-D-PRO-W" />
+      <xacro:arg name="base_frame" default="oak-d_frame" />
+      <xacro:arg name="parent_frame" default="oak-d-base-frame" />
+      <xacro:arg name="cam_pos_x" default="-0.0475" />
+      <xacro:arg name="cam_pos_y" default="0.13" />
+      <xacro:arg name="cam_pos_z" default="0.4465" />
+      <xacro:arg name="cam_roll" default="0.0" />
+      <xacro:arg name="cam_pitch" default="-1.5708" />
+      <xacro:arg name="cam_yaw" default="-1.5708" />
+      <xacro:arg name="rs_compat" default="false" />
+      <xacro:include filename="$(find trailblazer_description)/urdf/include/depthai_macro.xacro" />
+      <link name="$(arg parent_frame)" />
+      <xacro:depthai_camera camera_name="$(arg camera_name)" parent="$(arg parent_frame)"
+        camera_model="$(arg camera_model)" base_frame="$(arg base_frame)"
+        cam_pos_x="$(arg cam_pos_x)" cam_pos_y="$(arg cam_pos_y)" cam_pos_z="$(arg cam_pos_z)"
+        cam_roll="$(arg cam_roll)" cam_pitch="$(arg cam_pitch)" cam_yaw="$(arg cam_yaw)"
+        rs_compat="$(arg rs_compat)" />
+      <joint name="oakd_joint" type="fixed">
+          <parent link="chassis"/>
+          <child link="oak-d-base-frame"/>
+          <origin xyz="0 0 0" rpy="0 0 0"/>
+      </joint>
+      <!-- ******************************* OAK-D END ******************************* -->
   </xacro:if>
-  <xacro:unless value="$(arg use_ros2_control)">
+  <!-- <xacro:unless value="$(arg use_ros2_control)">
       <xacro:include filename="gazebo_control.xacro" />
-  </xacro:unless>
+      <xacro:include filename="depth_camera.xacro" />
+  </xacro:unless> -->
   <!-- ******************************* Links ******************************* -->
   <link name="base_link">

Commit message: ekf implementation

File: src/trailblazer_description/urdf/imu.xacro (robot description, xacro)
@@ -23,5 +23,5 @@
               </ros>
               <alwaysOn>true</alwaysOn>
-              <bodyName>base_footprint</bodyName>
+              <bodyName>base_link</bodyName>
               <topicName>imu</topicName>
               <serviceName>imu_service</serviceName>

File: src/trailblazer_description/urdf/rover.urdf.xacro (robot description, xacro)
@@ -42,11 +42,4 @@
   <link name="base_link">
   </link>
-  <joint name="base_footprint_joint" type="fixed">
-      <parent link="base_link"/>
-      <child link="base_footprint"/>
-      <origin xyz="0 0 0" rpy="0 0 0"/>
-  </joint>
-  <link name="base_footprint">
-  </link>
   <joint name="chassis_joint" type="fixed">
       <parent link="base_link"/>

Commit message: wheels to base_link

File: src/trailblazer_description/urdf/imu.xacro (robot description, xacro)
@@ -2,5 +2,5 @@
 <robot xmlns:xacro="http://www.ros.org/wiki/xacro">
     <joint name="imu_joint" type="fixed">
-        <parent link="chassis"/>
+        <parent link="base_link"/>
         <child link="imu_link"/>
         <origin xyz="0.001 0.146 0.4465" rpy="0 -1.5708 0"/>
@@ -19,46 +19,4 @@
         <always_on>true</always_on>
           <update_rate>200</update_rate>
-          <imu>
-            <angular_velocity>
-              <x>
-                <noise type="gaussian">
-                  <mean>0.0</mean>
-                  <stddev>2e-4</stddev>
-                </noise>
-              </x>
-              <y>
-                <noise type="gaussian">
-                  <mean>0.0</mean>
-                  <stddev>2e-4</stddev>
-                </noise>
-              </y>
-              <z>
-                <noise type="gaussian">
-                  <mean>0.0</mean>
-                  <stddev>2e-4</stddev>
-                </noise>
-              </z>
-            </angular_velocity>
-            <linear_acceleration>
-              <x>
-                <noise type="gaussian">
-                  <mean>0.0</mean>
-                  <stddev>1.7e-2</stddev>
-                </noise>
-              </x>
-              <y>
-                <noise type="gaussian">
-                  <mean>0.0</mean>
-                  <stddev>1.7e-2</stddev>
-                </noise>
-              </y>
-              <z>
-                <noise type="gaussian">
-                  <mean>0.0</mean>
-                  <stddev>1.7e-2</stddev>
-                </noise>
-              </z>
-            </linear_acceleration>
-          </imu>
            <plugin filename="libgazebo_ros_imu_sensor.so" name="imu_plugin">
               <initial_orientation_as_reference>false</initial_orientation_as_reference>

File: src/trailblazer_description/urdf/rover.urdf.xacro (robot description, xacro)
@@ -93,5 +93,5 @@
       <origin
         xyz="-0.0657932903439138 0.00142869200681425 9.9374601122415E-06"
-        rpy="0 0 0" />
+        rpy="0 0 1.5708" />
       <mass
         value="1.6444086136415" />
@@ -107,5 +107,5 @@
       <origin
         xyz="0 0 0"
-        rpy="0 0 0" />
+        rpy="0 0 3.14" />
       <geometry>
         <mesh
@@ -128,12 +128,14 @@
     </collision>
   </link>
+<!-- xyz="0.578691303668632 -0.237965989839832 0.501750000756599"  -->
+<!-- xyz="0.507691304 -0.540965989839832 0.121750000756599"  -->
   <joint
     name="FL_wheel_joint"
     type="continuous">
     <origin
-      xyz="0.578691303668632 -0.237965989839832 0.501750000756599"
-      rpy="0 0 0" />
+      xyz="0.501750000756599 -0.578691303668632 0.121750000756599"
+      rpy="0 0 1.5708" />
     <parent
-      link="chassis" />
+      link="base_link" />
     <child
       link="FL_wheel" />
@@ -174,5 +176,5 @@
       <origin
         xyz="0 0 0"
-        rpy="0 0 0" />
+        rpy="0 0 3.14" />
       <geometry>
         <mesh
@@ -185,8 +187,8 @@
     type="continuous">
     <origin
-      xyz="0.578691303668647 -0.237965989839099 -0.401750000000183"
-      rpy="0 0 0" />
+      xyz="-0.401750000756599 0.578691303668632 0.121750000756599"
+      rpy="0 0 1.5708" />
     <parent
-      link="chassis" />
+      link="base_link" />
     <child
       link="BL_wheel" />
@@ -213,5 +215,5 @@
       <origin
         xyz="0 0 0"
-        rpy="0 0 0" />
+        rpy="0 0 3.14" />
       <geometry>
         <mesh
@@ -238,8 +240,8 @@
     type="continuous">
     <origin
-      xyz="-0.578691303668549 -0.237965989839575 0.50175"
-      rpy="0 0 0" />
+      xyz="0.501750000756599 0.578691303668632 0.121750000756599"
+      rpy="0 0 1.57" />
     <parent
-      link="chassis" />
+      link="base_link" />
     <child
       link="FR_wheel" />
@@ -279,5 +281,5 @@
     <collision>
       <origin
-        xyz="0 0 0"
+        xyz="0 0 3.14"
         rpy="0 0 0" />
       <geometry>
@@ -291,8 +293,8 @@
     type="continuous">
     <origin
-      xyz="-0.578691303668548 -0.237965989839575 -0.401750000756777"
-      rpy="0 0 0" />
+      xyz="-0.401750000756599 -0.578691303668632 0.121750000756599"
+      rpy="0 0 1.57" />
     <parent
-      link="chassis" />
+      link="base_link" />
     <child
       link="BR_wheel" />
