Commit message: adding first test with wall_follower

File: src/trailblazer_description/urdf/lidar.xacro (robot description, xacro)
@@ -6,5 +6,5 @@
         <parent link="chassis"/>
         <child link="laser_frame"/>
-        <origin xyz="0.001 0.242 0.009" rpy="-1.5708 0 0"/>
+        <origin xyz="0.001 0.242 0.009" rpy="-1.5708 1.5708 0"/>
     </joint>
     <link name="laser_frame">
